Commit message: physical car assembled, running on its own now connected to laptop's WIFI hotspot

File: src/flipper_car/urdf/flipper_car.urdf (robot description, URDF)
Before this commit: robot flipper_car, 5 links, 4 joints
Links:
- link base_link: geometry collision box size=0.16 0.10 0.03; visual box size=0.015 0.09 0.032
